File: sticker.kicad_pcb (KiCad board)
At the start: 2 copper layers, 14.8 x 16.4 mm, 22 parts, among them U1 QFN, 48-Leads, Body 6,0x6,0mm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, X1 TSX-2520, X2 XTAL SMD 3.2 x 1.5 mm

Commit message: add schematic, symbols, export footprints, clean up
Parts:
- removed the C11 at (88.8, -83.0)
- removed the C11 at (78.3, -89.3)
- removed L6: Chip Inductor, 2-Leads, Body 1.0x0.5mm, IPC High Density, INDC1005X04L
- added C1: 12pF, dcdc:CAPC1005X04L, F.Cu at (87.5, -93.8)
- added C11: 100nF, dcdc:CAPC1005X04L, F.Cu at (79.7, -82.6)
- added L4: 10uH, dcdc:INDC1608X06L, F.Cu at (78.9, -87.5)
- added REF**: VIA-0.6096, dcdc:VIA-0.6096, F.Cu at (79.2, -93.6)
- added REF**: VIA-0.6096, dcdc:VIA-0.6096, F.Cu at (77.0, -79.6)
- added REF**: VIA-0.6096, dcdc:VIA-0.6096, F.Cu at (84.2, -93.1)
- added REF**: VIA-0.6096, dcdc:VIA-0.6096, F.Cu at (90.6, -81.7)
- added REF**: VIA-0.6096, dcdc:VIA-0.6096, F.Cu at (83.9, -91.1)
- added REF**: VIA-0.6096, dcdc:VIA-0.6096, F.Cu at (81.3, -82.4)
- added REF**: VIA-0.6096, dcdc:VIA-0.6096, F.Cu at (79.0, -82.1)
- added REF**: VIA-0.6096, dcdc:VIA-0.6096, F.Cu at (77.5, -90.9)
- added REF**: VIA-0.6096, dcdc:VIA-0.6096, F.Cu at (90.6, -89.4)
- added REF**: VIA-0.6096, dcdc:VIA-0.6096, F.Cu at (90.6, -91.3)
- added REF**: VIA-0.6096, dcdc:VIA-0.6096, F.Cu at (90.6, -79.6)
- added REF**: VIA-0.6096, dcdc:VIA-0.6096, F.Cu at (89.4, -94.1)
- added REF**: VIA-0.6096, dcdc:VIA-0.6096, F.Cu at (88.2, -79.6)
- added REF**: VIA-0.6096, dcdc:VIA-0.6096, F.Cu at (81.9, -79.6)
- added REF**: VIA-0.6096, dcdc:VIA-0.6096, F.Cu at (90.6, -87.3)
- added REF**: antenna, dcdc:antenna, F.Cu at (90.5, -90.4)
- added REF**: VIA-0.6096, dcdc:VIA-0.6096, F.Cu at (83.8, -94.8)
- added REF**: VIA-0.6096, dcdc:VIA-0.6096, F.Cu at (90.6, -94.8)
- added REF**: VIA-0.6096, dcdc:VIA-0.6096, F.Cu at (77.0, -94.8)
- added REF**: VIA-0.6096, dcdc:VIA-0.6096, F.Cu at (81.3, -94.8)
- added REF**: VIA-0.6096, dcdc:VIA-0.6096, F.Cu at (80.1, -90.9)
- added REF**: VIA-0.6096, dcdc:VIA-0.6096, F.Cu at (81.1, -88.8)
- added REF**: VIA-0.6096, dcdc:VIA-0.6096, F.Cu at (77.0, -83.1)
- C10: value Chip Capacitor, 2-Leads, Body 1.0x0.5mm, IPC High Density -> 47nF; footprint CAPC1005X04L -> dcdc:CAPC1005X04L
- C12: value Chip Capacitor, 2-Leads, Body 1.0x0.5mm, IPC High Density -> 1.0uF; footprint CAPC1005X04L -> dcdc:CAPC1608X06L
- C13, C14: footprint CAPC1005X04L -> dcdc:CAPC1005X04L
- C2: value Chip Capacitor, 2-Leads, Body 1.0x0.5mm, IPC High Density -> 12pF; footprint CAPC1005X04L -> dcdc:CAPC1005X04L
- C3: value Chip Capacitor, 2-Leads, Body 1.0x0.5mm, IPC High Density -> 2.2nF; footprint CAPC1005X04L -> dcdc:CAPC1005X04L
- C4: value Chip Capacitor, 2-Leads, Body 1.0x0.5mm, IPC High Density -> 1.0pF; footprint CAPC1005X04L -> dcdc:CAPC1005X04L
- C5: value Chip Capacitor, 2-Leads, Body 1.0x0.5mm, IPC High Density -> 3.9pF; footprint CAPC1005X04L -> dcdc:CAPC1005X04L
- C6: value Chip Capacitor, 2-Leads, Body 1.0x0.5mm, IPC High Density -> 1.5pF; footprint CAPC1005X04L -> dcdc:CAPC1005X04L
- C7: value Chip Capacitor, 2-Leads, Body 1.0x0.5mm, IPC High Density -> 4.7uF; footprint CAPC1005X04L -> dcdc:CAPC1608X06L
- C8: value Chip Capacitor, 2-Leads, Body 1.0x0.5mm, IPC High Density -> 100nF; footprint CAPC1005X04L -> dcdc:CAPC1005X04L
- C9: value Chip Capacitor, 2-Leads, Body 1.6x0.8mm, IPC High Density -> 1.0nF; footprint CAPC1608X06L -> dcdc:CAPC1005X04L
- L1: value Chip Inductor, 2-Leads, Body 1.0x0.5mm, IPC High Density -> 4.7nH; footprint INDC1005X04L -> dcdc:INDC1005X04L
- L2: value Chip Inductor, 2-Leads, Body 1.0x0.5mm, IPC High Density -> 27nH; footprint INDC1005X04L -> dcdc:INDC1005X04L
- L3: value Chip Inductor, 2-Leads, Body 1.0x0.5mm, IPC High Density -> 3.3nH; footprint INDC1005X04L -> dcdc:INDC1005X04L
- L5: value Chip Inductor, 2-Leads, Body 1.6x0.8mm, IPC High Density -> 15nH; footprint INDC1608X06L -> dcdc:INDC1005X04L
- U1: value QFN, 48-Leads, Body 6,0x6,0mm (max), Pitch 0,40mm, IPC Medium Density -> nrf51822-qfax; footprint QFN40P600X600X90-48N -> nrf:nrf51-qfax
- X1: value TSX-2520 -> Crystal; footprint BT-XTAL_2520 -> dcdc:BT-XTAL_2520
- X2: footprint XTAL_3215 -> dcdc:XTAL_3215
- moved C7 8.64 mm to (80.1, -89.3)
- moved C10 8.13 mm to (88.8, -83.0), turned to 180 degrees
- moved C9 7.33 mm to (87.4, -89.9), turned to 180 degrees
- moved C12 6.84 mm to (78.3, -89.3), turned to 180 degrees
- moved C8 2.55 mm to (84.8, -90.1), turned to 45 degrees
- moved L5 1.58 mm to (77.4, -87.9), turned to 180 degrees
- turned C2 to 225 degrees
- turned C4 to 90 degrees
- turned C6 to 180 degrees
- turned L1 to 180 degrees
- turned L2 to 180 degrees
- turned X1 to 180 degrees
Connections:
- net NetC6_1 renamed Net-(C6-Pad1)
- net P0.00 renamed Net-(U1-Pad4)
- net P0.01 renamed Net-(U1-Pad5)
- net P0.02 renamed Net-(U1-Pad6)
- net P0.03 renamed Net-(U1-Pad7)
- net P0.04 renamed Net-(U1-Pad8)
- net P0.05 renamed Net-(U1-Pad9)
- net P0.06 renamed Net-(U1-Pad10)
- net P0.07 renamed Net-(U1-Pad11)
- net P0.08 renamed Net-(U1-Pad14)
- net P0.09 renamed Net-(U1-Pad15)
- net P0.10 renamed Net-(U1-Pad16)
- net P0.11 renamed Net-(U1-Pad17)
- net P0.12 renamed Net-(U1-Pad18)
- net P0.13 renamed Net-(U1-Pad19)
- net P0.14 renamed Net-(U1-Pad20)
- net P0.15 renamed Net-(U1-Pad21)
- net P0.16 renamed Net-(U1-Pad22)
- net P0.17 renamed Net-(U1-Pad25)
- net P0.18 renamed Net-(U1-Pad26)
- net P0.19 renamed Net-(U1-Pad27)
- net P0.20 renamed Net-(U1-Pad28)
- net P0.21 renamed Net-(U1-Pad40)
- net P0.22 renamed Net-(U1-Pad41)
- net P0.23 renamed Net-(U1-Pad42)
- net P0.24 renamed Net-(U1-Pad43)
- net P0.25 renamed Net-(U1-Pad44)
- net P0.28 renamed Net-(U1-Pad47)
- net P0.29 renamed Net-(U1-Pad48)
- net P0.30 renamed Net-(U1-Pad3)
- net SWCLK renamed Net-(U1-Pad24)
- net SWDIO renamed Net-(U1-Pad23)
- C10 pad 1: NetC8_1 -> GND
- C10 pad 2: GND -> Net-(C10-Pad2)
- C12 pad 1: VCC_NRF -> Net-(C12-Pad1)
- C2 pad 1: NetC2_1 -> Net-(C2-Pad1)
- C3 pad 1: NetC3_1 -> Net-(C3-Pad1)
- C4 pad 1: NetC4_1 -> Net-(C4-Pad1)
- C5 pad 1: NetC5_1 -> Net-(C4-Pad1)
- C5 pad 2: NetC4_1 -> Net-(C5-Pad2)
- C7 pad 1: NetC1_1 -> Net-(C11-Pad1)
- C8 pad 1: AVDD -> GND
- C8 pad 2: GND -> Net-(C8-Pad2)
- C9 pad 1: VCC_NRF -> Net-(C12-Pad1)
- L1 pad 1: NetL1_1 -> Net-(C5-Pad2)
- L1 pad 2: NetC5_1 -> Net-(L1-Pad2)
- L2 pad 1: NetC3_1 -> Net-(L1-Pad2)
- L2 pad 2: NetL1_1 -> Net-(C3-Pad1)
- L3 pad 1: NetC4_1 -> Net-(C4-Pad1)
- L5 pad 1: NetL4_1 -> Net-(C12-Pad1)
- L5 pad 2: NetL4_2 -> Net-(L4-Pad1)
- U1 pad 1: VCC_NRF -> Net-(C11-Pad1)
- U1 pad 12: VCC_NRF -> Net-(C11-Pad1)
- U1 pad 2: NetL4_1 -> Net-(L4-Pad2)
- U1 pad 29: NetC10_1 -> Net-(C10-Pad2)
- U1 pad 30: NetC3_1 -> Net-(C3-Pad1)
- U1 pad 31: NetL1_1 -> Net-(L1-Pad2)
- U1 pad 32: NetC5_1 -> Net-(C5-Pad2)
- U1 pad 35: AVDD -> Net-(C12-Pad1)
- U1 pad 36: AVDD -> Net-(C12-Pad1)
- U1 pad 37: NetC1_1 -> Net-(C1-Pad1)
- U1 pad 38: NetC2_1 -> Net-(C2-Pad1)
- U1 pad 39: NetC8_1 -> Net-(C8-Pad2)
- U1 pad 45: XL2 -> Net-(U1-Pad45)
- U1 pad 46: XL1 -> Net-(U1-Pad46)
- X1 pad 1: NetC1_1 -> Net-(C2-Pad1)
- X1 pad 2: GND -> Net-(C1-Pad1)
- X1 pad 3: NetC2_1 -> GND
Routing:
- net (no net): track 100.2 -> 0.00 mm, vias 22 -> 0
- net Net-(C12-Pad1): track 0.00 -> 15.7 mm, vias 0 -> 2
- net AVDD: track 15.7 -> 0.00 mm, vias 2 -> 0
- net Net-(C11-Pad1): track 0.00 -> 11.2 mm, vias 0 -> 2
- net VCC_NRF: track 9.84 -> 0.00 mm, vias 2 -> 0
- net NetC1_1: track 6.86 -> 0.00 mm
- net Net-(C1-Pad1): track 0.00 -> 6.86 mm
- net Net-(C2-Pad1): track 0.00 -> 4.00 mm
- net NetC2_1: track 4.00 -> 0.00 mm
- net NetC3_1: track 3.56 -> 0.00 mm
- net Net-(C3-Pad1): track 0.00 -> 3.56 mm
- net NetC5_1: track 2.52 -> 0.00 mm
- net Net-(C5-Pad2): track 0.00 -> 2.52 mm
- net NetL1_1: track 2.45 -> 0.00 mm
- net Net-(L1-Pad2): track 0.00 -> 2.45 mm
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Other:
- net class Default: via_dia 0.889 -> 0.6096; via_drill 0.635 -> 0.3048
- net class Net-(C6-Pad1) added: clearance 0.1524, trace_width 0.9398, via_dia 0.6096, via_drill 0.3048
- rule trace_min: 0.254 -> 0.152
- rule via_min_drill: 0.508 -> 0.3048
- rule via_min_size: 0.889 -> 0.6096
